Commit message: fix little white urdf

File: unitree_robots/little_white/urdf/little_white.urdf (robot description, URDF)
Before this commit: robot littlewhite, 17 links, 16 joints
Joints:
- joint FL_calf_joint: limit lower=-2.7227 upper=-0.83776 effort=45.43 velocity=15.70 -> lower=-1.91 upper=0.0 effort=45.43 velocity=15.70
- joint FR_calf_joint: limit lower=-2.7227 upper=-0.83776 effort=45.43 velocity=15.70 -> lower=-1.91 upper=0.0 effort=45.43 velocity=15.70
- joint RL_calf_joint: limit lower=-2.7227 upper=-0.83776 effort=45.43 velocity=15.70 -> lower=-1.91 upper=0.0 effort=45.43 velocity=15.70
- joint RR_calf_joint: limit lower=-2.7227 upper=-0.83776 effort=45.43 velocity=15.70 -> lower=-1.91 upper=0.0 effort=45.43 velocity=15.70

Commit message: fix little white inertia and mass

File: unitree_robots/little_white/urdf/little_white.urdf (robot description, URDF)
Before this commit: robot littlewhite, 17 links, 16 joints
Links:
- link FL_calf_link: mass 0.499 -> 0.04
- link FL_hip_link: mass 1.188 -> 0.3
- link FL_thigh_link: mass 1.525 -> 0.48
- link FR_calf_link: mass 0.499 -> 0.04
- link FR_hip_link: mass 1.188 -> 0.3
- link FR_thigh_link: mass 1.525 -> 0.48
- link RL_calf_link: mass 0.499 -> 0.04
- link RL_hip_link: mass 1.188 -> 0.3
- link RL_thigh_link: mass 1.525 -> 0.48
- link RR_calf_link: mass 0.499 -> 0.04
- link RR_hip_link: mass 1.188 -> 0.3
- link RR_thigh_link: mass 1.525 -> 0.48
- link base_link: mass 6.512 -> 6.5

Commit message: fix little white urdf and mjcf

File: unitree_robots/little_white/urdf/little_white.urdf (robot description, URDF)
Before this commit: robot littlewhite, 17 links, 16 joints
Links:
- link base_link: mass 6.5 -> 2.0

Commit message: fix little white urdf and mjcf

File: unitree_robots/little_white/urdf/little_white.urdf (robot description, URDF)
Before this commit: robot littlewhite, 17 links, 16 joints
Joints:
- joint FL_thigh_joint: limit lower=-1.5708 upper=3.4907 effort=23.7 velocity=30.1 -> lower=-1.5708 upper=1.5708 effort=23.7 velocity=30.1
- joint FR_thigh_joint: limit lower=-1.5708 upper=3.4907 effort=23.7 velocity=30.1 -> lower=-1.5708 upper=1.5708 effort=23.7 velocity=30.1
- joint RL_thigh_joint: limit lower=-0.5236 upper=4.5379 effort=23.7 velocity=30.1 -> lower=-1.5708 upper=1.5708 effort=23.7 velocity=30.1
- joint RR_thigh_joint: limit lower=-0.5236 upper=4.5379 effort=23.7 velocity=30.1 -> lower=-1.5708 upper=1.5708 effort=23.7 velocity=30.1
