Commit message: fix(urdf): align g7_openarm joint limits and definitions with PinnZoo model

File: unitree_robots/g7_openarm/urdf/g7_openarm.urdf (robot description, URDF)
Before this commit: robot g7_openarm, 29 links, 28 joints
Links:
- added link L_gripper_tcp_link
- added link R_gripper_tcp_link
Joints:
- added joint L_gripper_tcp_joint: type fixed, parent L_link7, child L_gripper_tcp_link, origin xyz=0.000000 -0.031750 -0.189995 rpy=0 0 0
- added joint R_gripper_tcp_joint: type fixed, parent R_link7, child R_gripper_tcp_link, origin xyz=0.000000 0.031750 -0.189995 rpy=0 0 0
- joint AMR_FLW_joint: limit (none) -> effort=20 velocity=10
- joint AMR_FL_joint: limit (none) -> lower=-3.14159 upper=3.14159 effort=20 velocity=10
- joint AMR_FRW_joint: limit (none) -> effort=20 velocity=10
- joint AMR_FR_joint: limit (none) -> lower=-3.14159 upper=3.14159 effort=20 velocity=10
- joint AMR_RLW_joint: limit (none) -> effort=20 velocity=10
- joint AMR_RL_joint: limit (none) -> lower=-3.14159 upper=3.14159 effort=20 velocity=10
- joint AMR_RRW_joint: limit (none) -> effort=20 velocity=10
- joint AMR_RR_joint: limit (none) -> lower=-3.14159 upper=3.14159 effort=20 velocity=10
- joint L_1_joint: limit (none) -> lower=-1.3962629999999998 upper=3.490659 effort=40 velocity=16.754666
- joint L_2_joint: limit (none) -> lower=-0.17453267320510335 upper=3.3161253267948965 effort=40 velocity=16.754666
- joint L_3_joint: limit (none) -> lower=-1.570796 upper=1.570796 effort=27 velocity=5.445426
- joint L_4_joint: limit (none) -> lower=-2.443461 upper=0.0 effort=27 velocity=5.445426
- joint L_5_joint: limit (none) -> lower=-1.570796 upper=1.570796 effort=7 velocity=20.943946
- joint L_6_joint: limit lower=0 upper=0.09 effort=20 velocity=0.1 -> lower=-0.785398 upper=0.785398 effort=7 velocity=20.943946
- joint L_7_joint: limit (none) -> lower=-1.570796 upper=1.570796 effort=7 velocity=20.943946
- joint R_1_joint: limit (none) -> lower=-1.396263 upper=3.490659 effort=40 velocity=16.754666
- joint R_2_joint: limit (none) -> lower=-3.3161253267948965 upper=0.17453267320510335 effort=40 velocity=16.754666; type continuous -> revolute
- joint R_3_joint: limit (none) -> lower=-1.570796 upper=1.570796 effort=27 velocity=5.445426
- joint R_4_joint: limit (none) -> lower=-2.443461 upper=0.0 effort=27 velocity=5.445426
- joint R_5_joint: limit (none) -> lower=-1.570796 upper=1.570796 effort=7 velocity=20.943946
- joint R_6_joint: limit lower=0 upper=0.09 effort=20 velocity=0.1 -> lower=-0.785398 upper=0.785398 effort=7 velocity=20.943946
- joint R_7_joint: limit (none) -> lower=-1.570796 upper=1.570796 effort=7 velocity=20.943946
- joint gripper_LL_joint: axis 0 -1 0 -> 0 1 0; limit lower=0 upper=0.09 effort=20 velocity=0.1 -> lower=0.0 upper=0.045 effort=20 velocity=0.1; origin xyz=0 0.03075 -0.119 rpy=0 0 0 -> xyz=0 -0.01425 -0.119 rpy=0 0 0
- joint gripper_LR_joint: axis 0 1 0 -> 0 -1 0; limit lower=0 upper=0.09 effort=20 velocity=0.1 -> lower=0.0 upper=0.045 effort=20 velocity=0.1; origin xyz=0 -0.09425 -0.119 rpy=0 0 0 -> xyz=0 -0.04925 -0.119 rpy=0 0 0
- joint gripper_RL_joint: axis 0 -1 0 -> 0 1 0; limit lower=0 upper=0.09 effort=20 velocity=0.1 -> lower=0.0 upper=0.045 effort=20 velocity=0.1; origin xyz=0 0.09425 -0.119 rpy=0 0 0 -> xyz=0 0.04925 -0.119 rpy=0 0 0
- joint gripper_RR_joint: axis 0 1 0 -> 0 -1 0; limit lower=0 upper=0.09 effort=20 velocity=0.1 -> lower=0.0 upper=0.045 effort=20 velocity=0.1; origin xyz=0 -0.03075 -0.119 rpy=0 0 0 -> xyz=0 0.01425 -0.119 rpy=0 0 0
